Commit message: change robot model

File: src/vkc_example/env/env.urdf.xacro (robot description, xacro)
@@ -2,5 +2,6 @@
 <robot name="env" xmlns:xacro="http://ros.org/wiki/xacro">
   <!-- Includes -->
-  <xacro:include filename="$(find vkc_example)/urdf/deploy_husky_ur5e.urdf.xacro" />
+  <!-- <xacro:include filename="$(find vkc_example)/urdf/deploy_husky_ur5e.urdf.xacro" /> -->
+  <xacro:include filename="$(find vkc_example)/urdf/deploy_husky_ur5e_2f_85.urdf.xacro" />
   <!-- Arguments -->
   <xacro:arg name="husky_locx" default="0.0"/>

File: src/vkc_example/urdf/deploy_husky_ur5e_2f_85.urdf.xacro (robot description, xacro)
@@ -2,6 +2,4 @@
 <robot name="husky_ur5e_2f_85" xmlns:xacro="http://www.ros.org/wiki/xacro">
   <xacro:include filename="$(find husky_ur_description)/urdf/husky_ur5_e_description.urdf.xacro" />
-  <xacro:include filename="$(find robotiq_2f_85_gripper_visualization)/urdf/robotiq_arg2f_85_model_macro.xacro" />
-  <xacro:robotiq_arg2f_85 prefix="" />
   <joint name="2f_85_joint" type="fixed">
     <origin rpy="0.0 ${M_PI/2} 0" xyz="0.0 0.0 0.0" />
@@ -9,5 +7,5 @@
     <child link="robotiq_arg2f_base_link" />
   </joint>
-  <xacro:macro name="deploy" params="prefix attach_to_world loc_x loc_y orientation">
+  <xacro:macro name="deploy" params="prefix attach_to_world loc_x loc_y orientation has_gripper">
     <!-- Virtual Link Starts -->
     <link name="${prefix}virtual_base_x" />
@@ -43,4 +41,8 @@
       </joint>
     </xacro:if>
+    <xacro:if value="${has_gripper}">
+      <xacro:include filename="$(find robotiq_2f_85_gripper_visualization)/urdf/robotiq_arg2f_85_model_macro.xacro" />
+      <xacro:robotiq_arg2f_85 prefix="" />
+    </xacro:if>
   </xacro:macro>
 </robot>
