Commit message: set offset to ridgeback height

File: src/vkc_example/env/vkc_big_task.urdf.xacro (robot description, xacro)
@@ -40,5 +40,5 @@
     <parent link="world"/>
     <child link="$(arg robot_prefix)virtual_base_x"/>
-    <origin xyz="$(arg base_loc_x) $(arg base_loc_y) 0.0" rpy="0 0 $(arg base_loc_orient)" />
+    <origin xyz="$(arg base_loc_x) $(arg base_loc_y) 0.01965" rpy="0 0 $(arg base_loc_orient)" />
   </joint>
   <!-- ridgeback robot end -->

Commit message: update tieta srdf

File: src/vkc_example/env/vkc_big_task.urdf.xacro (robot description, xacro)
@@ -18,5 +18,5 @@
     <child link="base_link" />
     <axis xyz="0 0 1"/>
-    <limit effort="20" velocity="5.0" lower="-3.14" upper="3.14"/>
+    <limit effort="20" velocity="5.0" lower="-6.28" upper="6.28"/>
   </joint>
   <link name="$(arg robot_prefix)virtual_base_y"/>

Commit message: set joint limits for ridgeback ur

File: src/vkc_example/env/vkc_big_task.urdf.xacro (robot description, xacro)
@@ -18,5 +18,5 @@
     <child link="base_link" />
     <axis xyz="0 0 1"/>
-    <limit effort="20" velocity="5.0" lower="-6.28" upper="6.28"/>
+    <limit effort="20" velocity="5.0" lower="-3.14" upper="3.14"/>
   </joint>
   <link name="$(arg robot_prefix)virtual_base_y"/>

Commit message: feat: :boom: fixed base refactor to cartesian constraint

File: src/vkc_example/env/vkc_big_task.urdf.xacro (robot description, xacro)
@@ -14,4 +14,5 @@
   <link name="$(arg robot_prefix)virtual_base_theta"/>
   <joint name="$(arg robot_prefix)base_link_base_theta" type="revolute">
+  <!-- <joint name="$(arg robot_prefix)base_link_base_theta" type="continuous"> -->
     <parent link="$(arg robot_prefix)virtual_base_theta" />
     <origin xyz="0.0 0.0 0.0" rpy="0 0 0" />
@@ -19,4 +20,5 @@
     <axis xyz="0 0 1"/>
     <limit effort="20" velocity="5.0" lower="-3.14" upper="3.14"/>
+    <!-- <limit effort="20" velocity="5.0"/> -->
   </joint>
   <link name="$(arg robot_prefix)virtual_base_y"/>
