Commit message: vkc_big_task demo is included and a optional 3 finger gripper has provided to the other existing demos

File: src/robot_description/husky_ur_description/urdf/husky_ur5_e_description.urdf.xacro (robot description, xacro)
@@ -3,4 +3,6 @@
   <xacro:include filename="$(find ur_e_description)/urdf/ur5e.urdf.xacro" />
   <xacro:include filename="$(find husky_description)/urdf/husky.urdf.xacro" />
+  <!-- gripper -->
+  <xacro:include filename="$(find robotiq_3f_gripper_visualization)/cfg/robotiq-3f-gripper_articulated_macro.xacro" />
   <joint name="arm_mount_joint" type="fixed">
     <parent link="top_plate_link" />

File: src/robot_description/ridgeback_dual_arm_description/urdf/ridgeback_dual_arm.urdf.xacro (robot description, xacro)
@@ -19,11 +19,11 @@
   </joint>
   <!-- include pan tilt -->
-  <xacro:pan_tilt parent="base_footprint">
+  <!-- <xacro:pan_tilt parent="base_footprint">
     <origin xyz="0.25 0 1.02221" rpy="0 0 0"/>
-  </xacro:pan_tilt>
+  </xacro:pan_tilt> -->
   <!-- kinect dk -->
-  <xacro:kinect_dk parent="pan_tilt_surface">
+  <!-- <xacro:kinect_dk parent="pan_tilt_surface">
     <origin xyz="0 0 0" rpy="0 0 0"/>
-  </xacro:kinect_dk>
+  </xacro:kinect_dk> -->
   <!-- body -->
   <link name="body_link">
@@ -40,5 +40,5 @@
       <origin xyz="0.25 0.68 0" rpy="0 0 0"/>
       <geometry>
-        <box size="0.16 0.46 0.2"/>
+        <box size="0.16 0.70 0.2"/>
       </geometry>
     </collision>

File: src/robot_description/robotiq_3f_gripper_visualization/cfg/robotiq-3f-gripper_finger_articulated_macro.xacro (robot description, xacro)
@@ -18,5 +18,4 @@
 				</material>
 			</visual>
-		<!--
 			<collision>
 				<origin xyz="0.020 0 0" rpy="0 0 0"/>
@@ -28,5 +27,4 @@
 				</material>
 			</collision>
-        -->
             <inertial>
                 <origin xyz="0 0 0" rpy="0 0 0"/>
@@ -43,5 +41,4 @@
 				<material name="gray"/>
 			</visual>
-		<!--
 			<collision>
 				<origin xyz="0.050 -.028 0" rpy="0 0 -0.52"/>
@@ -51,5 +48,4 @@
 				<material name="yellow"/>
 			</collision>
-		-->
             <inertial>
                 <origin xyz="0 0 0" rpy="0 0 0"/>
@@ -71,5 +67,4 @@
 				<material name="gray"/>
 			</visual>
-		<!--
 			<collision>
 				<origin xyz="0.039 0 0.0075" rpy="0 0 0"/>
@@ -79,5 +74,4 @@
 				<material name="yellow"/>
 			</collision>
-		-->
             <inertial>
                 <origin xyz="0 0 0" rpy="0 0 0"/>
@@ -94,5 +88,4 @@
 				<material name="gray"/>
 			</visual>
-		<!--
 			<collision>
 				<origin xyz="0 0 0" rpy="0 0 0.52"/>
@@ -102,5 +95,4 @@
 				<material name="yellow"/>
 			</collision>
-		-->
             <inertial>
                 <origin xyz="0 0 0" rpy="0 0 0"/>

File: src/vkc_example/env/env.urdf.xacro (robot description, xacro)
@@ -7,4 +7,5 @@
   <xacro:arg name="husky_locy" default="0.0"/>
   <xacro:arg name="husky_orient" default="0.0"/>
+  <xacro:arg name="has_gripper" default="true"/>
   <xacro:property name="rigid_mesh_dir" value="package://scene_builder/output/vkc_demo/assets/rigid" />
   <!-- <link name="ground">
@@ -41,4 +42,4 @@
   <!-- Setup Environment -->
   <link name="world"/>
-  <xacro:deploy prefix="" attach_to_world="true" loc_x="$(arg husky_locx)" loc_y="$(arg husky_locy)" orientation="$(arg husky_orient)" />
+  <xacro:deploy prefix="" attach_to_world="true" loc_x="$(arg husky_locx)" loc_y="$(arg husky_locy)" orientation="$(arg husky_orient)" has_gripper="$(arg has_gripper)"/>
 </robot>

File: src/vkc_example/env/vkc_demo.urdf.xacro (robot description, xacro)
@@ -2,47 +2,4 @@
 <robot xmlns:xacro="http://ros.org/wiki/xacro" name="scene">
   <!-- <xacro:include filename="$(find scene_builder)/output/vkc_demo/main.xacro" /> -->
-  <!-- <xacro:include filename="$(find vkc_example)/urdf/deploy_husky_ur5e.urdf.xacro" /> -->
- <!-- ridgeback robot begin -->
-  <!-- <xacro:include filename="$(find ridgeback_dual_arm_description)/urdf/ridgeback_dual_arm.urdf.xacro" /> -->
-  <!-- Arguments -->
-  <!-- <xacro:arg name="base_locx" default="0.0"/>
-  <xacro:arg name="base_locy" default="0.0"/>
-  <xacro:arg name="base_orient" default="0.0"/>
-  <xacro:arg name="robot_prefix" default=""/> -->
-  <!-- Setup Environment -->
-  <!--
-    link order: world link -> virtual_base_x -> virtual_base_y -> virtual_base_theta -> base_link
-  -->
-  <!-- <link name="$(arg robot_prefix)virtual_base_theta"/>
-  <joint name="$(arg robot_prefix)base_link_base_theta" type="revolute">
-    <parent link="$(arg robot_prefix)virtual_base_theta" />
-    <origin xyz="0.0 0.0 0.0" rpy="0 0 0" />
-    <child link="base_link" />
-    <axis xyz="0 0 1"/>
-    <limit effort="20" velocity="5.0" lower="-3.14" upper="3.14"/>
-  </joint>
-  <link name="$(arg robot_prefix)virtual_base_y"/>
-  <joint name="$(arg robot_prefix)base_theta_base_y" type="prismatic">
-    <parent link="$(arg robot_prefix)virtual_base_y" />
-    <origin xyz="0.0 0.0 0.0" rpy="0 0 0" />
-    <child link="$(arg robot_prefix)virtual_base_theta" />
-    <axis xyz="0 1 0"/>
-    <limit effort="20" velocity="5.0" lower="-10" upper="10"/>
-  </joint>
-  <link name="$(arg robot_prefix)virtual_base_x"/>
-  <joint name="$(arg robot_prefix)base_y_base_x" type="prismatic">
-    <parent link="$(arg robot_prefix)virtual_base_x" />
-    <origin xyz="0.0 0.0 0.0" rpy="0 0 0" />
-    <child link="$(arg robot_prefix)virtual_base_y" />
-    <axis xyz="1 0 0"/>
-    <limit effort="20" velocity="5.0" lower="-10" upper="10"/>
-  </joint>
-  <link name="world"/>
-  <joint name="world_to_base_footprint" type="fixed">
-    <origin xyz="0 0 0" rpy="0 0 0"/>
-    <parent link="world"/>
-    <child link="$(arg robot_prefix)virtual_base_x"/>
-  </joint> -->
-  <!-- ridgeback robot end -->
   <xacro:include filename="$(find vkc_example)/urdf/deploy_husky_ur5e.urdf.xacro" />
   <!-- Arguments -->
@@ -50,6 +7,7 @@
   <xacro:arg name="husky_locy" default="0.0"/>
   <xacro:arg name="husky_orient" default="0.0"/>
+  <xacro:arg name="has_gripper" default="true"/>
   <!-- Setup Environment -->
   <link name="world"/>
-  <xacro:deploy prefix="" attach_to_world="true" loc_x="$(arg husky_locx)" loc_y="$(arg husky_locy)" orientation="$(arg husky_orient)" />
+  <xacro:deploy prefix="" attach_to_world="true" loc_x="$(arg husky_locx)" loc_y="$(arg husky_locy)" orientation="$(arg husky_orient)"  has_gripper="$(arg has_gripper)"/>
 </robot>

File: src/vkc_example/urdf/deploy_husky_ur5e.urdf.xacro (robot description, xacro)
@@ -2,5 +2,5 @@
 <robot xmlns:xacro="http://www.ros.org/wiki/xacro">
   <xacro:include filename="$(find husky_ur_description)/urdf/husky_ur5_e_description.urdf.xacro" />
-  <xacro:macro name="deploy" params="prefix attach_to_world loc_x loc_y orientation">
+  <xacro:macro name="deploy" params="prefix attach_to_world loc_x loc_y orientation has_gripper">
     <!-- Virtual Link Starts -->
     <link name="${prefix}virtual_base_x">
@@ -66,4 +66,36 @@
       </joint>
     </xacro:if>
+    <xacro:if value="${has_gripper}">
+      <!-- gipper flange -->
+      <link name="gripper_flange">
+        <visual>
+          <origin xyz="0 0 0" rpy="0 0 0"/>
+          <geometry>
+            <mesh filename="package://husky_ur_description/meshes/3-finger-gripper_fixed-urdf.stl"/>
+          </geometry>
+          <material name="">
+            <color rgba="0.2 0.2 0.2 1"/>
+          </material>
+        </visual>
+        <collision>
+          <origin xyz="0 0 0" rpy="0 0 0"/>
+          <geometry>
+            <mesh filename="package://husky_ur_description/meshes/3-finger-gripper_fixed-urdf.stl"/>
+          </geometry>
+        </collision>
+      </link>
+      <joint name="gripper_flange_joint" type="fixed">
+          <origin xyz="0 0 0" rpy="0 0 0"/>
+          <parent link="ur_arm_tool0"/>
+          <child link="gripper_flange"/>
+      </joint>
+      <!-- gripper -->
+      <xacro:robotiq-3f-gripper_articulated prefix="gripper_"/>
+      <joint name="gripper_joint" type="fixed">
+          <origin xyz="0 0 0.068825" rpy="${M_PI/2} 0 0"/>
+          <parent link="gripper_flange"/>
+          <child link="gripper_palm"/>
+      </joint>
+    </xacro:if>
   </xacro:macro>
 </robot>
