Commit message: for pog exp

File: src/robot_description/husky_description/urdf/decorations.urdf.xacro (robot description, xacro)
@@ -121,10 +121,10 @@
             </geometry>
           </visual>
-          <collision>
+          <!-- <collision>
             <origin xyz="0 0 0" rpy="0 0 0"/>
             <geometry>
               <mesh filename="package://husky_description/meshes/large_top_plate_collision.stl" />
             </geometry>
-          </collision>
+          </collision> -->
         </link>
         <!-- Attach top plate -->
@@ -155,10 +155,10 @@
             </geometry>
           </visual>
-          <collision>
+          <!-- <collision>
             <origin xyz="0 0 0" rpy="0 0 0"/>
             <geometry>
               <mesh filename="package://husky_description/meshes/top_plate.dae" />
             </geometry>
-          </collision>
+          </collision> -->
         </link>
         <!-- Attach top plate -->

File: src/robot_description/husky_description/urdf/husky.urdf.xacro (robot description, xacro)
@@ -63,14 +63,14 @@
       <origin xyz="0 0 0.05" rpy="0 0 0" />
       <geometry>
-      <!-- <cylinder radius="0.5" length="0.3"/> -->
-        <box size="${ base_x_size + husky_front_bumper_extend + husky_rear_bumper_extend } ${base_y_size} ${base_z_size/2}"/>
+      <cylinder radius="0.5" length="0.3"/>
+        <!-- <box size="${ base_x_size + husky_front_bumper_extend + husky_rear_bumper_extend } ${base_y_size} ${base_z_size/2}"/> -->
       </geometry>
     </collision>
-    <collision>
+    <!-- <collision>
       <origin xyz="0 0 ${base_z_size*3/4-0.01}" rpy="0 0 0" />
       <geometry>
         <box size="${base_x_size*4/5} ${base_y_size} ${base_z_size/2-0.02}"/>
       </geometry>
-    </collision>
+    </collision> -->
   </link>
   <!-- Base footprint is on the ground under the robot -->

File: src/robot_description/husky_description/urdf/wheel.urdf.xacro (robot description, xacro)
@@ -49,5 +49,5 @@
 			<fdir1 value="1 0 0"/>
 		</gazebo>
-		<joint name="${wheel_prefix}_wheel" type="continuous">
+		<joint name="${wheel_prefix}_wheel" type="fixed">
 			<parent link="base_link"/>
 			<child link="${wheel_prefix}_wheel_link"/>

File: src/robot_description/ur_e_description/urdf/ur5e.urdf.xacro (robot description, xacro)
@@ -7,11 +7,9 @@
       <mass value="${mass}" />
       <xacro:insert_block name="origin" />
-      <inertia ixx="${0.0833333 * mass * (3 * radius * radius + length * length)}" ixy="0.0" ixz="0.0"
-        iyy="${0.0833333 * mass * (3 * radius * radius + length * length)}" iyz="0.0"
-        izz="${0.5 * mass * radius * radius}" />
+      <inertia ixx="${0.0833333 * mass * (3 * radius * radius + length * length)}" ixy="0.0" ixz="0.0" iyy="${0.0833333 * mass * (3 * radius * radius + length * length)}" iyz="0.0" izz="${0.5 * mass * radius * radius}" />
     </inertial>
   </xacro:macro>
   <xacro:macro name="ur5e_robot" params="prefix joint_limited
-    shoulder_pan_lower_limit:=${-pi}    shoulder_pan_upper_limit:=${pi}
+    shoulder_pan_lower_limit:=${-2*pi}    shoulder_pan_upper_limit:=${2*pi}
     shoulder_lift_lower_limit:=${-pi}    shoulder_lift_upper_limit:=${pi}
     elbow_joint_lower_limit:=${-pi}    elbow_joint_upper_limit:=${pi}
@@ -23,5 +21,5 @@
     safety_k_position:=20">
     <!-- Inertia parameters -->
-    <xacro:property name="base_mass" value="4.0" />  <!-- This mass might be incorrect -->
+    <xacro:property name="base_mass" value="4.0" /> <!-- This mass might be incorrect -->
     <xacro:property name="shoulder_mass" value="3.7000" />
     <xacro:property name="upper_arm_mass" value="8.3930" />
@@ -65,17 +63,21 @@
     <xacro:property name="wrist_3_length" value="${d6}" />
     <!--property name="shoulder_height" value="0.089159" /-->
-    <!--property name="shoulder_offset" value="0.13585" /-->  <!-- shoulder_offset - elbow_offset + wrist_1_length = 0.10915 -->
+    <!--property name="shoulder_offset" value="0.13585" /-->
+    <!-- shoulder_offset - elbow_offset + wrist_1_length = 0.10915 -->
     <!--property name="upper_arm_length" value="0.42500" /-->
-    <!--property name="elbow_offset" value="0.1197" /-->       <!-- CAD measured -->
+    <!--property name="elbow_offset" value="0.1197" /-->
+    <!-- CAD measured -->
     <!--property name="forearm_length" value="0.39225" /-->
-    <!--property name="wrist_1_length" value="0.093" /-->     <!-- CAD measured -->
-    <!--property name="wrist_2_length" value="0.09465" /-->   <!-- In CAD this distance is 0.930, but in the spec it is 0.09465 -->
+    <!--property name="wrist_1_length" value="0.093" /-->
+    <!-- CAD measured -->
+    <!--property name="wrist_2_length" value="0.09465" /-->
+    <!-- In CAD this distance is 0.930, but in the spec it is 0.09465 -->
     <!--property name="wrist_3_length" value="0.0823" /-->
-    <xacro:property name="shoulder_radius" value="0.060" />   <!-- manually measured -->
-    <xacro:property name="upper_arm_radius" value="0.054" />  <!-- manually measured -->
-    <xacro:property name="elbow_radius" value="0.060" />      <!-- manually measured -->
-    <xacro:property name="forearm_radius" value="0.040" />    <!-- manually measured -->
-    <xacro:property name="wrist_radius" value="0.045" />      <!-- manually measured -->
-    <link name="${prefix}base_link" >
+    <xacro:property name="shoulder_radius" value="0.060" /> <!-- manually measured -->
+    <xacro:property name="upper_arm_radius" value="0.054" /> <!-- manually measured -->
+    <xacro:property name="elbow_radius" value="0.060" /> <!-- manually measured -->
+    <xacro:property name="forearm_radius" value="0.040" /> <!-- manually measured -->
+    <xacro:property name="wrist_radius" value="0.045" /> <!-- manually measured -->
+    <link name="${prefix}base_link">
       <visual>
         <geometry>
@@ -83,5 +85,5 @@
         </geometry>
         <material name="LightGrey">
-          <color rgba="0.7 0.7 0.7 1.0"/>
+          <color rgba="0.7 0.7 0.7 1.0" />
         </material>
       </visual>
@@ -97,20 +99,20 @@
     <joint name="${prefix}shoulder_pan_joint" type="revolute">
       <parent link="${prefix}base_link" />
-      <child link = "${prefix}shoulder_link" />
+      <child link="${prefix}shoulder_link" />
       <origin xyz="0.0 0.0 ${shoulder_height}" rpy="0.0 0.0 0.0" />
       <axis xyz="0 0 1" />
       <xacro:unless value="${joint_limited}">
-        <limit lower="${-2.0 * pi}" upper="${2.0 * pi}" effort="150.0" velocity="3.14"/>
-        <xacro:if value="${safety_limits}">
-          <safety_controller soft_lower_limit="${-2.0 * pi + safety_pos_margin}" soft_upper_limit="${2.0 * pi - safety_pos_margin}" k_position="${safety_k_position}" k_velocity="0.0"/>
-        </xacro:if>
-      </xacro:unless>
-      <xacro:if value="${joint_limited}">
-        <limit lower="${shoulder_pan_lower_limit}" upper="${shoulder_pan_upper_limit}" effort="150.0" velocity="3.14"/>
-        <xacro:if value="${safety_limits}">
-          <safety_controller soft_lower_limit="${shoulder_pan_lower_limit + safety_pos_margin}" soft_upper_limit="${shoulder_pan_upper_limit - safety_pos_margin}" k_position="${safety_k_position}" k_velocity="0.0"/>
-        </xacro:if>
-      </xacro:if>
-      <dynamics damping="0.0" friction="0.0"/>
+        <limit lower="${-2.0 * pi}" upper="${2.0 * pi}" effort="150.0" velocity="3.14" />
+        <xacro:if value="${safety_limits}">
+          <safety_controller soft_lower_limit="${-2.0 * pi + safety_pos_margin}" soft_upper_limit="${2.0 * pi - safety_pos_margin}" k_position="${safety_k_position}" k_velocity="0.0" />
+        </xacro:if>
+      </xacro:unless>
+      <xacro:if value="${joint_limited}">
+        <limit lower="${shoulder_pan_lower_limit}" upper="${shoulder_pan_upper_limit}" effort="150.0" velocity="3.14" />
+        <xacro:if value="${safety_limits}">
+          <safety_controller soft_lower_limit="${shoulder_pan_lower_limit + safety_pos_margin}" soft_upper_limit="${shoulder_pan_upper_limit - safety_pos_margin}" k_position="${safety_k_position}" k_velocity="0.0" />
+        </xacro:if>
+      </xacro:if>
+      <dynamics damping="0.0" friction="0.0" />
     </joint>
     <link name="${prefix}shoulder_link">
@@ -120,5 +122,5 @@
         </geometry>
         <material name="LightGrey">
-          <color rgba="0.7 0.7 0.7 1.0"/>
+          <color rgba="0.7 0.7 0.7 1.0" />
         </material>
       </visual>
@@ -134,20 +136,20 @@
     <joint name="${prefix}shoulder_lift_joint" type="revolute">
       <parent link="${prefix}shoulder_link" />
-      <child link = "${prefix}upper_arm_link" />
+      <child link="${prefix}upper_arm_link" />
       <origin xyz="0.0 ${shoulder_offset} 0.0" rpy="0.0 ${pi / 2.0} 0.0" />
       <axis xyz="0 1 0" />
       <xacro:unless value="${joint_limited}">
-        <limit lower="${-2.0 * pi}" upper="${2.0 * pi}" effort="150.0" velocity="3.14"/>
-        <xacro:if value="${safety_limits}">
-          <safety_controller soft_lower_limit="${-2.0 * pi + safety_pos_margin}" soft_upper_limit="${2.0 * pi - safety_pos_margin}" k_position="${safety_k_position}" k_velocity="0.0"/>
-        </xacro:if>
-      </xacro:unless>
-      <xacro:if value="${joint_limited}">
-        <limit lower="${shoulder_lift_lower_limit}" upper="${shoulder_lift_upper_limit}" effort="150.0" velocity="3.14"/>
-        <xacro:if value="${safety_limits}">
-          <safety_controller soft_lower_limit="${shoulder_lift_lower_limit + safety_pos_margin}" soft_upper_limit="${shoulder_lift_upper_limit - safety_pos_margin}" k_position="${safety_k_position}" k_velocity="0.0"/>
-        </xacro:if>
-      </xacro:if>
-      <dynamics damping="0.0" friction="0.0"/>
+        <limit lower="${-2.0 * pi}" upper="${2.0 * pi}" effort="150.0" velocity="3.14" />
+        <xacro:if value="${safety_limits}">
+          <safety_controller soft_lower_limit="${-2.0 * pi + safety_pos_margin}" soft_upper_limit="${2.0 * pi - safety_pos_margin}" k_position="${safety_k_position}" k_velocity="0.0" />
+        </xacro:if>
+      </xacro:unless>
+      <xacro:if value="${joint_limited}">
+        <limit lower="${shoulder_lift_lower_limit}" upper="${shoulder_lift_upper_limit}" effort="150.0" velocity="3.14" />
+        <xacro:if value="${safety_limits}">
+          <safety_controller soft_lower_limit="${shoulder_lift_lower_limit + safety_pos_margin}" soft_upper_limit="${shoulder_lift_upper_limit - safety_pos_margin}" k_position="${safety_k_position}" k_velocity="0.0" />
+        </xacro:if>
+      </xacro:if>
+      <dynamics damping="0.0" friction="0.0" />
     </joint>
     <link name="${prefix}upper_arm_link">
@@ -157,5 +159,5 @@
         </geometry>
         <material name="LightGrey">
-          <color rgba="0.7 0.7 0.7 1.0"/>
+          <color rgba="0.7 0.7 0.7 1.0" />
         </material>
       </visual>
@@ -171,20 +173,20 @@
     <joint name="${prefix}elbow_joint" type="revolute">
       <parent link="${prefix}upper_arm_link" />
-      <child link = "${prefix}forearm_link" />
+      <child link="${prefix}forearm_link" />
       <origin xyz="0.0 ${elbow_offset} ${upper_arm_length}" rpy="0.0 0.0 0.0" />
       <axis xyz="0 1 0" />
       <xacro:unless value="${joint_limited}">
-        <limit lower="${-pi}" upper="${pi}" effort="150.0" velocity="3.14"/>
-        <xacro:if value="${safety_limits}">
-          <safety_controller soft_lower_limit="${-2.0 * pi + safety_pos_margin}" soft_upper_limit="${2.0 * pi - safety_pos_margin}" k_position="${safety_k_position}" k_velocity="0.0"/>
-        </xacro:if>
-      </xacro:unless>
-      <xacro:if value="${joint_limited}">
-        <limit lower="${elbow_joint_lower_limit}" upper="${elbow_joint_upper_limit}" effort="150.0" velocity="3.14"/>
-        <xacro:if value="${safety_limits}">
-          <safety_controller soft_lower_limit="${elbow_joint_lower_limit + safety_pos_margin}" soft_upper_limit="${elbow_joint_upper_limit - safety_pos_margin}" k_position="${safety_k_position}" k_velocity="0.0"/>
-        </xacro:if>
-      </xacro:if>
-      <dynamics damping="0.0" friction="0.0"/>
+        <limit lower="${-pi}" upper="${pi}" effort="150.0" velocity="3.14" />
+        <xacro:if value="${safety_limits}">
+          <safety_controller soft_lower_limit="${-2.0 * pi + safety_pos_margin}" soft_upper_limit="${2.0 * pi - safety_pos_margin}" k_position="${safety_k_position}" k_velocity="0.0" />
+        </xacro:if>
+      </xacro:unless>
+      <xacro:if value="${joint_limited}">
+        <limit lower="${elbow_joint_lower_limit}" upper="${elbow_joint_upper_limit}" effort="150.0" velocity="3.14" />
+        <xacro:if value="${safety_limits}">
+          <safety_controller soft_lower_limit="${elbow_joint_lower_limit + safety_pos_margin}" soft_upper_limit="${elbow_joint_upper_limit - safety_pos_margin}" k_position="${safety_k_position}" k_velocity="0.0" />
+        </xacro:if>
+      </xacro:if>
+      <dynamics damping="0.0" friction="0.0" />
     </joint>
     <link name="${prefix}forearm_link">
@@ -194,5 +196,5 @@
         </geometry>
         <material name="LightGrey">
-          <color rgba="0.7 0.7 0.7 1.0"/>
+          <color rgba="0.7 0.7 0.7 1.0" />
         </material>
       </visual>
@@ -208,20 +210,20 @@
     <joint name="${prefix}wrist_1_joint" type="revolute">
       <parent link="${prefix}forearm_link" />
-      <child link = "${prefix}wrist_1_link" />
+      <child link="${prefix}wrist_1_link" />
       <origin xyz="0.0 0.0 ${forearm_length}" rpy="0.0 ${pi / 2.0} 0.0" />
       <axis xyz="0 1 0" />
       <xacro:unless value="${joint_limited}">
-        <limit lower="${-2.0 * pi}" upper="${2.0 * pi}" effort="28.0" velocity="6.28"/>
-        <xacro:if value="${safety_limits}">
-          <safety_controller soft_lower_limit="${-2.0 * pi + safety_pos_margin}" soft_upper_limit="${2.0 * pi - safety_pos_margin}" k_position="${safety_k_position}" k_velocity="0.0"/>
-        </xacro:if>
-      </xacro:unless>
-      <xacro:if value="${joint_limited}">
-        <limit lower="${wrist_1_lower_limit}" upper="${wrist_1_upper_limit}" effort="28.0" velocity="6.28"/>
-        <xacro:if value="${safety_limits}">
-          <safety_controller soft_lower_limit="${wrist_1_lower_limit + safety_pos_margin}" soft_upper_limit="${wrist_1_upper_limit - safety_pos_margin}" k_position="${safety_k_position}" k_velocity="0.0"/>
-        </xacro:if>
-      </xacro:if>
-      <dynamics damping="0.0" friction="0.0"/>
+        <limit lower="${-2.0 * pi}" upper="${2.0 * pi}" effort="28.0" velocity="6.28" />
+        <xacro:if value="${safety_limits}">
+          <safety_controller soft_lower_limit="${-2.0 * pi + safety_pos_margin}" soft_upper_limit="${2.0 * pi - safety_pos_margin}" k_position="${safety_k_position}" k_velocity="0.0" />
+        </xacro:if>
+      </xacro:unless>
+      <xacro:if value="${joint_limited}">
+        <limit lower="${wrist_1_lower_limit}" upper="${wrist_1_upper_limit}" effort="28.0" velocity="6.28" />
+        <xacro:if value="${safety_limits}">
+          <safety_controller soft_lower_limit="${wrist_1_lower_limit + safety_pos_margin}" soft_upper_limit="${wrist_1_upper_limit - safety_pos_margin}" k_position="${safety_k_position}" k_velocity="0.0" />
+        </xacro:if>
+      </xacro:if>
+      <dynamics damping="0.0" friction="0.0" />
     </joint>
     <link name="${prefix}wrist_1_link">
@@ -231,5 +233,5 @@
         </geometry>
         <material name="LightGrey">
-          <color rgba="0.7 0.7 0.7 1.0"/>
+          <color rgba="0.7 0.7 0.7 1.0" />
         </material>
       </visual>
@@ -245,20 +247,20 @@
     <joint name="${prefix}wrist_2_joint" type="revolute">
       <parent link="${prefix}wrist_1_link" />
-      <child link = "${prefix}wrist_2_link" />
+      <child link="${prefix}wrist_2_link" />
       <origin xyz="0.0 ${wrist_1_length} 0.0" rpy="0.0 0.0 0.0" />
       <axis xyz="0 0 1" />
       <xacro:unless value="${joint_limited}">
-        <limit lower="${-2.0 * pi}" upper="${2.0 * pi}" effort="28.0" velocity="6.28"/>
-        <xacro:if value="${safety_limits}">
-          <safety_controller soft_lower_limit="${-2.0 * pi + safety_pos_margin}" soft_upper_limit="${2.0 * pi - safety_pos_margin}" k_position="${safety_k_position}" k_velocity="0.0"/>
-        </xacro:if>
-      </xacro:unless>
-      <xacro:if value="${joint_limited}">
-        <limit lower="${wrist_2_lower_limit}" upper="${wrist_2_upper_limit}" effort="28.0" velocity="6.28"/>
-        <xacro:if value="${safety_limits}">
-          <safety_controller soft_lower_limit="${wrist_2_lower_limit + safety_pos_margin}" soft_upper_limit="${wrist_2_upper_limit - safety_pos_margin}" k_position="${safety_k_position}" k_velocity="0.0"/>
-        </xacro:if>
-      </xacro:if>
-      <dynamics damping="0.0" friction="0.0"/>
+        <limit lower="${-2.0 * pi}" upper="${2.0 * pi}" effort="28.0" velocity="6.28" />
+        <xacro:if value="${safety_limits}">
+          <safety_controller soft_lower_limit="${-2.0 * pi + safety_pos_margin}" soft_upper_limit="${2.0 * pi - safety_pos_margin}" k_position="${safety_k_position}" k_velocity="0.0" />
+        </xacro:if>
+      </xacro:unless>
+      <xacro:if value="${joint_limited}">
+        <limit lower="${wrist_2_lower_limit}" upper="${wrist_2_upper_limit}" effort="28.0" velocity="6.28" />
+        <xacro:if value="${safety_limits}">
+          <safety_controller soft_lower_limit="${wrist_2_lower_limit + safety_pos_margin}" soft_upper_limit="${wrist_2_upper_limit - safety_pos_margin}" k_position="${safety_k_position}" k_velocity="0.0" />
+        </xacro:if>
+      </xacro:if>
+      <dynamics damping="0.0" friction="0.0" />
     </joint>
     <link name="${prefix}wrist_2_link">
@@ -268,5 +270,5 @@
         </geometry>
         <material name="LightGrey">
-          <color rgba="0.7 0.7 0.7 1.0"/>
+          <color rgba="0.7 0.7 0.7 1.0" />
         </material>
       </visual>
@@ -282,21 +284,21 @@
     <joint name="${prefix}wrist_3_joint" type="revolute">
       <parent link="${prefix}wrist_2_link" />
-      <child link = "${prefix}wrist_3_link" />
+      <child link="${prefix}wrist_3_link" />
       <origin xyz="0.0 0.0 ${wrist_2_length}" rpy="0.0 0.0 0.0" />
       <axis xyz="0 1 0" />
       <xacro:unless value="${joint_limited}">
-        <limit lower="${-2.0 * pi}" upper="${2.0 * pi}" effort="28.0" velocity="6.28"/>
-        <xacro:if value="${safety_limits}">
-          <safety_controller soft_lower_limit="${-2.0 * pi + safety_pos_margin}" soft_upper_limit="${2.0 * pi - safety_pos_margin}" k_position="${safety_k_position}" k_velocity="0.0"/>
-        </xacro:if>
-      </xacro:unless>
-      <xacro:if value="${joint_limited}">
-        <limit lower="${-2.0 * pi}" upper="${2.0 * pi}" effort="28.0" velocity="6.28"/>
+        <limit lower="${-2.0 * pi}" upper="${2.0 * pi}" effort="28.0" velocity="6.28" />
+        <xacro:if value="${safety_limits}">
+          <safety_controller soft_lower_limit="${-2.0 * pi + safety_pos_margin}" soft_upper_limit="${2.0 * pi - safety_pos_margin}" k_position="${safety_k_position}" k_velocity="0.0" />
+        </xacro:if>
+      </xacro:unless>
+      <xacro:if value="${joint_limited}">
+        <limit lower="${-2.0 * pi}" upper="${2.0 * pi}" effort="28.0" velocity="6.28" />
         <!-- <limit lower="${wrist_3_lower_limit}" upper="${wrist_3_upper_limit}" effort="28.0" velocity="6.28"/> -->
         <xacro:if value="${safety_limits}">
-          <safety_controller soft_lower_limit="${wrist_3_lower_limit + safety_pos_margin}" soft_upper_limit="${wrist_3_upper_limit - safety_pos_margin}" k_position="${safety_k_position}" k_velocity="0.0"/>
-        </xacro:if>
-      </xacro:if>
-      <dynamics damping="0.0" friction="0.0"/>
+          <safety_controller soft_lower_limit="${wrist_3_lower_limit + safety_pos_margin}" soft_upper_limit="${wrist_3_upper_limit - safety_pos_margin}" k_position="${safety_k_position}" k_velocity="0.0" />
+        </xacro:if>
+      </xacro:if>
+      <dynamics damping="0.0" friction="0.0" />
     </joint>
     <link name="${prefix}wrist_3_link">
@@ -306,5 +308,5 @@
         </geometry>
         <material name="LightGrey">
-          <color rgba="0.7 0.7 0.7 1.0"/>
+          <color rgba="0.7 0.7 0.7 1.0" />
         </material>
       </visual>
@@ -320,5 +322,5 @@
     <joint name="${prefix}ee_fixed_joint" type="fixed">
       <parent link="${prefix}wrist_3_link" />
-      <child link = "${prefix}ee_link" />
+      <child link="${prefix}ee_link" />
       <origin xyz="0.0 ${wrist_3_length} 0.0" rpy="0.0 0.0 ${pi/2.0}" />
     </joint>
@@ -326,7 +328,7 @@
       <collision>
         <geometry>
-          <box size="0.01 0.01 0.01"/>
-        </geometry>
-        <origin rpy="0 0 0" xyz="-0.01 0 0"/>
+          <box size="0.01 0.01 0.01" />
+        </geometry>
+        <origin rpy="0 0 0" xyz="-0.01 0 0" />
       </collision>
     </link>
@@ -334,5 +336,5 @@
     <xacro:ur_arm_gazebo prefix="${prefix}" />
     <!-- ROS base_link to UR 'Base' Coordinates transform -->
-    <link name="${prefix}base"/>
+    <link name="${prefix}base" />
     <joint name="${prefix}base_link-base_fixed_joint" type="fixed">
       <!-- NOTE: this rotation is only needed as long as base_link itself is
@@ -340,14 +342,20 @@
                  degrees)
       -->
-      <origin xyz="0 0 0" rpy="0 0 ${-pi}"/>
-      <parent link="${prefix}base_link"/>
-      <child link="${prefix}base"/>
+      <origin xyz="0 0 0" rpy="0 0 ${-pi}" />
+      <parent link="${prefix}base_link" />
+      <child link="${prefix}base" />
     </joint>
     <!-- Frame coincident with all-zeros TCP on UR controller -->
-    <link name="${prefix}tool0"/>
+    <!-- <link name="${prefix}tool0"/>
     <joint name="${prefix}wrist_3_link-tool0_fixed_joint" type="fixed">
       <origin xyz="0 ${wrist_3_length} 0" rpy="${pi/-2.0} 0 0"/>
       <parent link="${prefix}wrist_3_link"/>
       <child link="${prefix}tool0"/>
+    </joint> -->
+    <link name="${prefix}tool0" />
+    <joint name="${prefix}ee_link-tool0_fixed_joint" type="fixed">
+      <origin rpy="0. 1.57 1.57" xyz="0.20 0.0 0.0" />
+      <parent link="${prefix}ee_link" />
+      <child link="${prefix}tool0" />
     </joint>
   </xacro:macro>
