Commit message: refine arena_env node to disable rotation of husky and playback the refined trajectory instead

File: src/robot_description/husky_description/urdf/husky.urdf.xacro (robot description, xacro)
@@ -63,6 +63,6 @@
       <origin xyz="0 0 0.05" rpy="0 0 0" />
       <geometry>
-      <cylinder radius="0.5" length="0.3"/>
-        <!-- <box size="${ base_x_size + husky_front_bumper_extend + husky_rear_bumper_extend } ${base_y_size} ${base_z_size/2}"/> -->
+      <!-- <cylinder radius="0.5" length="0.3"/> -->
+        <box size="${ base_x_size + husky_front_bumper_extend + husky_rear_bumper_extend } ${base_y_size} ${base_z_size/2}"/>
       </geometry>
     </collision>

Commit message: run open door experiment for mujoco simulation

File: src/robot_description/husky_description/urdf/husky.urdf.xacro (robot description, xacro)
@@ -60,17 +60,17 @@
     </visual>
     <collision>
-      <!-- <origin xyz="${( husky_front_bumper_extend - husky_rear_bumper_extend ) / 2.0} 0 ${base_z_size/4}" rpy="0 0 0" /> -->
+      <origin xyz="${( husky_front_bumper_extend - husky_rear_bumper_extend ) / 2.0} 0 ${base_z_size/4}" rpy="0 0 0" />
       <origin xyz="0 0 0.05" rpy="0 0 0" />
       <geometry>
-      <cylinder radius="0.5" length="0.3"/>
-        <!-- <box size="${ base_x_size + husky_front_bumper_extend + husky_rear_bumper_extend } ${base_y_size} ${base_z_size/2}"/> -->
+      <!-- <cylinder radius="0.5" length="0.3"/> -->
+        <box size="${ base_x_size + husky_front_bumper_extend + husky_rear_bumper_extend } ${base_y_size} ${base_z_size/2}"/>
       </geometry>
     </collision>
-    <!-- <collision>
+    <collision>
       <origin xyz="0 0 ${base_z_size*3/4-0.01}" rpy="0 0 0" />
       <geometry>
         <box size="${base_x_size*4/5} ${base_y_size} ${base_z_size/2-0.02}"/>
       </geometry>
-    </collision> -->
+    </collision>
   </link>
   <!-- Base footprint is on the ground under the robot -->

File: src/robot_description/ur_e_description/urdf/ur5e.urdf.xacro (robot description, xacro)
@@ -11,5 +11,5 @@
   </xacro:macro>
   <xacro:macro name="ur5e_robot" params="prefix joint_limited
-    shoulder_pan_lower_limit:=${-2*pi}    shoulder_pan_upper_limit:=${2*pi}
+    shoulder_pan_lower_limit:=${-pi}    shoulder_pan_upper_limit:=${pi}
     shoulder_lift_lower_limit:=${-pi}    shoulder_lift_upper_limit:=${pi}
     elbow_joint_lower_limit:=${-pi}    elbow_joint_upper_limit:=${pi}

File: src/vkc_example/urdf/deploy_husky_ur5e_2f_85.urdf.xacro (robot description, xacro)
@@ -40,5 +40,5 @@
         <child link="${prefix}virtual_base_x" />
         <parent link="world" />
-        <origin xyz="${loc_x} ${loc_y} 0.20" rpy="0 0 ${orientation}" />
+        <origin xyz="${loc_x} ${loc_y} 0.145" rpy="0 0 ${orientation}" />
       </joint>
     </xacro:if>

Commit message: enlarge wheel size for safe planning

File: src/robot_description/husky_description/urdf/husky.urdf.xacro (robot description, xacro)
@@ -49,5 +49,6 @@
   <xacro:property name="wheel_vertical_offset" value="0.03282" />
   <!-- Wheel Properties -->
-  <xacro:property name="wheel_length" value="0.1143" />
+  <!-- 0.1143 -->
+  <xacro:property name="wheel_length" value="0.15" />
   <xacro:property name="wheel_radius" value="0.1651" />
   <!-- Base link is the center of the robot's bottom plate -->

Commit message: modify husky ur5 model

File: src/robot_description/husky_description/urdf/husky.urdf.xacro (robot description, xacro)
@@ -64,14 +64,14 @@
       <origin xyz="0 0 0.05" rpy="0 0 0" />
       <geometry>
-      <!-- <cylinder radius="0.5" length="0.3"/> -->
-        <box size="${ base_x_size + husky_front_bumper_extend + husky_rear_bumper_extend } ${base_y_size} ${base_z_size/2}"/>
+      <cylinder radius="0.5" length="0.3"/>
+        <!-- <box size="${ base_x_size + husky_front_bumper_extend + husky_rear_bumper_extend } ${base_y_size} ${base_z_size/2}"/> -->
       </geometry>
     </collision>
-    <collision>
+    <!-- <collision>
       <origin xyz="0 0 ${base_z_size*3/4-0.01}" rpy="0 0 0" />
       <geometry>
         <box size="${base_x_size*4/5} ${base_y_size} ${base_z_size/2-0.02}"/>
       </geometry>
-    </collision>
+    </collision> -->
   </link>
   <!-- Base footprint is on the ground under the robot -->

File: src/robot_description/husky_description/urdf/wheel.urdf.xacro (robot description, xacro)
@@ -35,10 +35,10 @@
 				</geometry>
 			</visual>
-			<collision>
+			<!-- <collision>
 				<origin xyz="0 0 0" rpy="${M_PI/2} 0 0" />
 				<geometry>
 					<cylinder length="${wheel_length}" radius="${wheel_radius}" />
 				</geometry>
-			</collision>
+			</collision> -->
 		</link>
 		<gazebo reference="${wheel_prefix}_wheel_link">

Commit message: feat: save current work

File: src/robot_description/husky_description/urdf/husky.urdf.xacro (robot description, xacro)
@@ -64,5 +64,5 @@
       <origin xyz="0 0 0.05" rpy="0 0 0" />
       <geometry>
-      <cylinder radius="0.5" length="0.3"/>
+      <cylinder radius="0.1" length="0.3"/>
         <!-- <box size="${ base_x_size + husky_front_bumper_extend + husky_rear_bumper_extend } ${base_y_size} ${base_z_size/2}"/> -->
       </geometry>

Commit message: add sr env

File: src/robot_description/husky_description/urdf/husky.urdf.xacro (robot description, xacro)
@@ -64,5 +64,5 @@
       <origin xyz="0 0 0.05" rpy="0 0 0" />
       <geometry>
-      <cylinder radius="0.1" length="0.3"/>
+      <cylinder radius="0.5" length="0.3"/>
         <!-- <box size="${ base_x_size + husky_front_bumper_extend + husky_rear_bumper_extend } ${base_y_size} ${base_z_size/2}"/> -->
       </geometry>

Commit message: update attach locations in household env

File: src/robot_description/husky_description/urdf/husky.urdf.xacro (robot description, xacro)
@@ -64,6 +64,6 @@
       <origin xyz="0 0 0.05" rpy="0 0 0" />
       <geometry>
-      <cylinder radius="0.5" length="0.3"/>
-        <!-- <box size="${ base_x_size + husky_front_bumper_extend + husky_rear_bumper_extend } ${base_y_size} ${base_z_size/2}"/> -->
+      <cylinder radius="0.47" length="0.4"/>
+        <!-- <box size="${ base_x_size + husky_front_bumper_extend + husky_rear_bumper_extend } ${base_y_size+wheel_length} ${base_z_size/2}"/> -->
       </geometry>
     </collision>

File: src/robot_description/ur_e_description/urdf/ur5e.urdf.xacro (robot description, xacro)
@@ -11,5 +11,5 @@
   </xacro:macro>
   <xacro:macro name="ur5e_robot" params="prefix joint_limited
-    shoulder_pan_lower_limit:=${-pi}    shoulder_pan_upper_limit:=${pi}
+    shoulder_pan_lower_limit:=${-2.*pi}    shoulder_pan_upper_limit:=${2.*pi}
     shoulder_lift_lower_limit:=${-pi}    shoulder_lift_upper_limit:=${pi}
     elbow_joint_lower_limit:=${-pi}    elbow_joint_upper_limit:=${pi}
@@ -294,6 +294,6 @@
       </xacro:unless>
       <xacro:if value="${joint_limited}">
-        <limit lower="${-2.0 * pi}" upper="${2.0 * pi}" effort="28.0" velocity="6.28" />
-        <!-- <limit lower="${wrist_3_lower_limit}" upper="${wrist_3_upper_limit}" effort="28.0" velocity="6.28"/> -->
+        <!-- <limit lower="${-2.0 * pi}" upper="${2.0 * pi}" effort="28.0" velocity="6.28" /> -->
+        <limit lower="${wrist_3_lower_limit}" upper="${wrist_3_upper_limit}" effort="28.0" velocity="6.28"/>
         <xacro:if value="${safety_limits}">
           <safety_controller soft_lower_limit="${wrist_3_lower_limit + safety_pos_margin}" soft_upper_limit="${wrist_3_upper_limit - safety_pos_margin}" k_position="${safety_k_position}" k_velocity="0.0" />
