Commit message: refine trajectory

File: src/robot_description/robotiq_2f_85_gripper_visualization/urdf/robotiq_arg2f_85_model_macro.xacro (robot description, xacro)
@@ -130,5 +130,5 @@
   </xacro:macro>
   <xacro:macro name="inner_knuckle_joint" params="prefix fingerprefix reflect">
-    <joint name="${prefix}${fingerprefix}_inner_knuckle_joint" type="revolute">
+    <joint name="${prefix}${fingerprefix}_inner_knuckle_joint" type="fixed">
       <!-- <origin xyz="0 ${reflect * -0.0127} 0.06142" rpy="${pi / 2 + .725} 0 ${(reflect - 1) * pi / 2}" /> -->
       <origin xyz="0 ${reflect * -0.0127} 0.06142" rpy="0 0 ${(1 + reflect) * pi / 2}"/>
@@ -141,5 +141,5 @@
   </xacro:macro>
   <xacro:macro name="inner_finger_joint" params="prefix fingerprefix">
-    <joint name="${prefix}${fingerprefix}_inner_finger_joint" type="revolute">
+    <joint name="${prefix}${fingerprefix}_inner_finger_joint" type="fixed">
       <origin xyz="0 0.0061 0.0471" rpy="0 0 0"/>
       <parent link="${prefix}${fingerprefix}_outer_finger" />
@@ -160,5 +160,5 @@
   <xacro:include filename="$(find robotiq_2f_85_gripper_visualization)/urdf/robotiq_arg2f.xacro" />
   <xacro:macro name="finger_joint" params="prefix">
-    <joint name="${prefix}finger_joint" type="revolute">
+    <joint name="${prefix}finger_joint" type="fixed">
       <origin xyz="0 -0.0306011 0.054904" rpy="0 0 ${pi}"/>
       <parent link="${prefix}robotiq_arg2f_base_link" />
@@ -170,5 +170,5 @@
   </xacro:macro>
   <xacro:macro name="right_outer_knuckle_joint" params="prefix">
-    <joint name="${prefix}right_outer_knuckle_joint" type="revolute">
+    <joint name="${prefix}right_outer_knuckle_joint" type="fixed">
       <origin xyz="0 0.0306011 0.054904" rpy="0 0 0"/>
       <parent link="${prefix}robotiq_arg2f_base_link" />

File: src/vkc_example/urdf/deploy_husky_ur5e_2f_85.urdf.xacro (robot description, xacro)
@@ -18,5 +18,5 @@
       <child link="base_link" />
       <axis xyz="0 0 1" />
-      <limit effort="20" velocity="5.0" lower="-3.14" upper="3.14" />
+      <limit effort="20" velocity="5.0" lower="-6.28" upper="6.28" />
     </joint>
     <joint name="${prefix}base_theta_base_y" type="prismatic">
