Commit message: uam env long horizon task

File: src/robot_description/aerialvkc_v3000_description/urdf/aerialvkc_v3000_description_simplify.urdf.xacro (robot description, xacro)
@@ -561,9 +561,10 @@
     </collision>
   </link>
-  <joint name="arm_joint_I" type="continuous">
+  <joint name="arm_joint_I" type="revolute">
     <origin xyz="0 -0.0171000000000001 -0.0640000000000012" rpy="-1.5707963267949 1.5707963267949 3.14159265358979" />
     <parent link="base_link" />
     <child link="arm_link_I" />
     <axis xyz="0 0 -1" />
+    <limit effort="30" lower="-1.57" upper="1.57" velocity="10" />
   </joint>
   <link name="arm_link_II">
@@ -588,9 +589,10 @@
     </collision>
   </link>
-  <joint name="arm_joint_II" type="continuous">
+  <joint name="arm_joint_II" type="revolute">
     <origin xyz="0.0795000000000011 0 0.000599999999999989" rpy="3.14159265358979 0 0" />
     <parent link="arm_link_I" />
     <child link="arm_link_II" />
     <axis xyz="0 0 1" />
+    <limit effort="30" lower="-1.57" upper="1.57" velocity="10" />
   </joint>
   <link name="gripper_base_link">
@@ -615,9 +617,10 @@
     </collision>
   </link>
-  <joint name="gripper_base_joint" type="continuous">
+  <joint name="gripper_base_joint" type="revolute">
     <origin xyz="0.081 0 0.0115" rpy="1.58355301227902 0 3.14159265358979" />
     <parent link="arm_link_II" />
     <child link="gripper_base_link" />
     <axis xyz="1 0 0" />
+    <limit effort="30" lower="-3.14" upper="3.14" velocity="10" />
   </joint>
   <link name="gear_arm_link_I">

File: src/vkc_example/env/uam_env.xacro (robot description, xacro)
@@ -2,8 +2,9 @@
 <robot xmlns:xacro="http://ros.org/wiki/xacro" name="uam_env">
   <xacro:include filename="$(find vkc_example)/urdf/deploy_uam.urdf.xacro" />
+  <!-- <xacro:include filename="$(find scene_builder)/output/uam_env/main.xacro" /> -->
   <!-- Arguments -->
   <xacro:arg name="x" default="0.0"/>
   <xacro:arg name="y" default="0.0"/>
-  <xacro:arg name="z" default="0.5"/>
+  <xacro:arg name="z" default="0.0"/>
   <!-- Setup Environment -->
   <link name="world"/>
