Commit message: feat: added tieta env

File: src/robot_description/robotiq_3f_gripper_visualization/cfg/robotiq-3f-gripper_finger_articulated_macro.xacro (robot description, xacro)
@@ -18,5 +18,5 @@
 				</material>
 			</visual>
-			<!-- <collision>
+			<collision>
 				<origin xyz="0.020 0 0" rpy="0 0 0"/>
 				<geometry>
@@ -26,5 +26,5 @@
 					<color rgba="0 1 1 1"/>
 				</material>
-			</collision> -->
+			</collision>
             <inertial>
                 <origin xyz="0 0 0" rpy="0 0 0"/>
@@ -67,5 +67,5 @@
 				<material name="gray"/>
 			</visual>
-			<!-- <collision>
+			<collision>
 				<origin xyz="0.039 0 0.0075" rpy="0 0 0"/>
 				<geometry>
@@ -73,5 +73,5 @@
 				</geometry>
 				<material name="yellow"/>
-			</collision> -->
+			</collision>
             <inertial>
                 <origin xyz="0 0 0" rpy="0 0 0"/>
@@ -88,5 +88,5 @@
 				<material name="gray"/>
 			</visual>
-			<!-- <collision>
+			<collision>
 				<origin xyz="0 0 0" rpy="0 0 0.52"/>
 				<geometry>
@@ -94,5 +94,5 @@
 				</geometry>
 				<material name="yellow"/>
-			</collision> -->
+			</collision>
             <inertial>
                 <origin xyz="0 0 0" rpy="0 0 0"/>
