Commit message: complete functional(tool, container, articulated object) implementation with partly collision disabled

File: src/robot_description/ridgeback_dual_arm_description/urdf/ridgeback_dual_arm.urdf.xacro (robot description, xacro)
@@ -37,4 +37,10 @@
       </material>
     </visual>
+    <collision>
+      <origin xyz="0.25 0.68 0" rpy="0 0 0"/>
+      <geometry>
+        <box size="0.16 0.46 0.2"/>
+      </geometry>
+    </collision>
   </link>
   <joint name="body_joint" type="fixed">

Commit message: the complete demo sequence passed test

File: src/robot_description/ridgeback_dual_arm_description/urdf/ridgeback_dual_arm.urdf.xacro (robot description, xacro)
@@ -19,11 +19,11 @@
   </joint>
   <!-- include pan tilt -->
-  <!-- <xacro:pan_tilt parent="base_footprint">
+  <xacro:pan_tilt parent="base_footprint">
     <origin xyz="0.25 0 1.02221" rpy="0 0 0"/>
-  </xacro:pan_tilt> -->
+  </xacro:pan_tilt>
   <!-- kinect dk -->
-  <!-- <xacro:kinect_dk parent="pan_tilt_surface">
+  <xacro:kinect_dk parent="pan_tilt_surface">
     <origin xyz="0 0 0" rpy="0 0 0"/>
-  </xacro:kinect_dk> -->
+  </xacro:kinect_dk>
   <!-- body -->
   <link name="body_link">
@@ -98,4 +98,10 @@
       </material>
     </visual>
+    <collision>
+      <origin xyz="0 0 0" rpy="0 0 0"/>
+      <geometry>
+        <mesh filename="package://ridgeback_dual_arm_description/mesh/3-finger-gripper_fixed-urdf.stl"/>
+      </geometry>
+    </collision>
   </link>
   <joint name="right_gripper_flange_joint" type="fixed">

Commit message: add ridgeback dual arm

File: src/robot_description/ridgeback_dual_arm_description/urdf/ridgeback_dual_arm.urdf.xacro (robot description, xacro)
@@ -50,12 +50,12 @@
   </joint>
   <!-- left arm -->
-  <!-- <xacro:ur5e_robot prefix="left_arm_" />
+  <xacro:ur5e_robot prefix="left_arm_" />
   <joint name="left_arm_joint" type="fixed">
       <origin xyz="0.25 0.208336 0.957336" rpy="-${M_PI/4*3} 0 0"/>
       <parent link="base_footprint"/>
       <child link="left_arm_base_link"/>
-  </joint> -->
+  </joint>
   <!-- left gipper flange -->
-  <!-- <link name="left_gripper_flange">
+  <link name="left_gripper_flange">
     <visual>
       <origin xyz="0 0 0" rpy="0 0 0"/>
@@ -72,21 +72,21 @@
       <parent link="left_arm_tool0"/>
       <child link="left_gripper_flange"/>
-  </joint> -->
+  </joint>
   <!-- left gripper -->
-  <!-- <xacro:robotiq-3f-gripper_articulated prefix="left_gripper_"/>
+  <xacro:robotiq-3f-gripper_articulated prefix="left_gripper_"/>
   <joint name="left_gripper_joint" type="fixed">
       <origin xyz="0 0 0.068825" rpy="${M_PI/2} 0 0"/>
       <parent link="left_gripper_flange"/>
       <child link="left_gripper_palm"/>
-  </joint> -->
+  </joint>
   <!-- right arm -->
-  <xacro:ur5e_robot prefix="right_arm_" />
+  <!-- <xacro:ur5e_robot prefix="right_arm_" />
   <joint name="right_arm_joint" type="fixed">
       <origin xyz="0.25 -0.208336 0.957336" rpy="${M_PI/4*3} 0 0"/>
       <parent link="base_footprint"/>
       <child link="right_arm_base_link"/>
-  </joint>
+  </joint> -->
   <!-- right gipper flange -->
-  <link name="right_gripper_flange">
+  <!-- <link name="right_gripper_flange">
     <visual>
       <origin xyz="0 0 0" rpy="0 0 0"/>
@@ -109,11 +109,11 @@
       <parent link="right_arm_tool0"/>
       <child link="right_gripper_flange"/>
-  </joint>
+  </joint> -->
   <!-- right gripper -->
-  <xacro:robotiq-3f-gripper_articulated prefix="right_gripper_"/>
+  <!-- <xacro:robotiq-3f-gripper_articulated prefix="right_gripper_"/>
   <joint name="right_gripper_joint" type="fixed">
       <origin xyz="0 0 0.068825" rpy="${M_PI/2} 0 0"/>
       <parent link="right_gripper_flange"/>
       <child link="right_gripper_palm"/>
-  </joint>
+  </joint>   -->
 </robot>

File: src/robot_description/robotiq_3f_gripper_visualization/cfg/robotiq-3f-gripper_finger_articulated_macro.xacro (robot description, xacro)
@@ -18,5 +18,5 @@
 				</material>
 			</visual>
-			<collision>
+			<!-- <collision>
 				<origin xyz="0.020 0 0" rpy="0 0 0"/>
 				<geometry>
@@ -26,5 +26,5 @@
 					<color rgba="0 1 1 1"/>
 				</material>
-			</collision>
+			</collision> -->
             <inertial>
                 <origin xyz="0 0 0" rpy="0 0 0"/>
@@ -41,5 +41,5 @@
 				<material name="gray"/>
 			</visual>
-			<collision>
+			<!-- <collision>
 				<origin xyz="0.050 -.028 0" rpy="0 0 -0.52"/>
 				<geometry>
@@ -47,5 +47,5 @@
 				</geometry>
 				<material name="yellow"/>
-			</collision>
+			</collision> -->
             <inertial>
                 <origin xyz="0 0 0" rpy="0 0 0"/>
@@ -67,5 +67,5 @@
 				<material name="gray"/>
 			</visual>
-			<collision>
+			<!-- <collision>
 				<origin xyz="0.039 0 0.0075" rpy="0 0 0"/>
 				<geometry>
@@ -73,5 +73,5 @@
 				</geometry>
 				<material name="yellow"/>
-			</collision>
+			</collision> -->
             <inertial>
                 <origin xyz="0 0 0" rpy="0 0 0"/>
@@ -88,5 +88,5 @@
 				<material name="gray"/>
 			</visual>
-			<collision>
+			<!-- <collision>
 				<origin xyz="0 0 0" rpy="0 0 0.52"/>
 				<geometry>
@@ -94,5 +94,5 @@
 				</geometry>
 				<material name="yellow"/>
-			</collision>
+			</collision> -->
             <inertial>
                 <origin xyz="0 0 0" rpy="0 0 0"/>

File: src/vkc_example/env/vkc_big_task.urdf.xacro (robot description, xacro)
@@ -6,5 +6,5 @@
   <xacro:arg name="base_loc_x" default="0.0"/>
   <xacro:arg name="base_loc_y" default="0.0"/>
-  <xacro:arg name="base_loc_orient" default="1.57"/>
+  <xacro:arg name="base_loc_orient" default="0.0"/>
   <xacro:arg name="robot_prefix" default=""/>
   <!-- Setup Environment -->

Commit message: fix ridgeback urdf

File: src/robot_description/ridgeback_dual_arm_description/urdf/ridgeback_dual_arm.urdf.xacro (robot description, xacro)
@@ -1,20 +1,20 @@
 <?xml version="1.0"?>
 <robot name="ridgeback_dual_arm" xmlns:xacro="http://www.ros.org/wiki/xacro">
-  <xacro:property name="M_PI" value="3.1415926535897931"/>
+  <xacro:property name="M_PI" value="3.1415926535897931" />
   <!-- include ridgeback -->
-  <xacro:include filename="$(find ridgeback_description)/urdf/ridgeback.urdf.xacro"/>
+  <xacro:include filename="$(find ridgeback_description)/urdf/ridgeback.urdf.xacro" />
   <!-- include ur 5e arm -->
-  <xacro:include filename="$(find ur_description)/urdf/inc/ur5e_macro.xacro"/>
+  <xacro:include filename="$(find ur_description)/urdf/inc/ur5e_macro.xacro" />
   <!-- include kinect dk -->
-  <xacro:include filename="$(find ridgeback_dual_arm_description)/urdf/kinect_dk.xacro"/>
+  <xacro:include filename="$(find ridgeback_dual_arm_description)/urdf/kinect_dk.xacro" />
   <!-- include pan tilt -->
-  <xacro:include filename="$(find pan_tilt_description)/urdf/pan_tilt.urdf.xacro"/>
+  <xacro:include filename="$(find pan_tilt_description)/urdf/pan_tilt.urdf.xacro" />
   <!-- gripper -->
   <xacro:include filename="$(find robotiq_3f_gripper_visualization)/cfg/robotiq-3f-gripper_articulated_macro.xacro" />
   <link name="base_footprint" />
   <joint name="footprint_joint" type="fixed">
-      <origin xyz="0 0 -0.01965" rpy="0 0 0"/>
-      <parent link="base_link"/>
-      <child link="base_footprint"/>
+    <origin xyz="0 0 -0.01965" rpy="0 0 0" />
+    <parent link="base_link" />
+    <child link="base_footprint" />
   </joint>
   <!-- include pan tilt -->
@@ -29,54 +29,67 @@
   <link name="body_link">
     <visual>
-      <origin xyz="0 0 0" rpy="0 0 0"/>
+      <origin xyz="0 0 0" rpy="0 0 0" />
       <geometry>
-        <mesh filename="package://ridgeback_dual_arm_description/mesh/ridgeback_2xur5-sup-simp-urdf.stl"/>
+        <!-- <mesh filename="package://ridgeback_dual_arm_description/mesh/ridgeback_2xur5-sup-simp-urdf.stl"/> -->
+        <mesh filename="package://ridgeback_dual_arm_description/mesh/ridgeback-2xur5e-all-urdf.stl" />
       </geometry>
       <material name="">
-        <color rgba="0.2 0.2 0.2 1"/>
+        <color rgba="0.2 0.2 0.2 1" />
       </material>
     </visual>
     <collision>
-      <origin xyz="0.25 0.68 0" rpy="0 0 0"/>
+      <origin xyz="0 0 0" rpy="0 0 0" />
       <geometry>
-        <box size="0.16 0.70 0.2"/>
+        <mesh filename="package://ridgeback_dual_arm_description/mesh/ridgeback-2xur5e-all-urdf.stl" />
       </geometry>
     </collision>
   </link>
   <joint name="body_joint" type="fixed">
-      <origin xyz="0 0 0" rpy="${M_PI/2} 0 0"/>
-      <parent link="base_footprint"/>
-      <child link="body_link"/>
+    <origin xyz="0 0 0" rpy="0 0 0" />
+    <parent link="base_footprint" />
+    <child link="body_link" />
+  </joint>
+  <!-- left_body -->
+  <link name="left_body_link" />
+  <joint name="left_body_joint" type="fixed">
+    <origin xyz="0.2 0.22 1.233" rpy="${M_PI/4*3} 0 0" />
+    <parent link="base_footprint" />
+    <child link="left_body_link" />
   </joint>
   <!-- left arm -->
   <xacro:ur5e_robot prefix="left_arm_" />
-  <joint name="left_arm_joint" type="fixed">
+  <!-- <joint name="left_arm_joint" type="fixed">
       <origin xyz="0.25 0.208336 0.957336" rpy="-${M_PI/4*3} 0 0"/>
       <parent link="base_footprint"/>
       <child link="left_arm_base_link"/>
+  </joint> -->
+  <joint name="left_arm_joint" type="fixed">
+    <origin xyz="0 0 0" rpy="${M_PI/2} ${M_PI/2} 0" />
+    <parent link="left_body_link" />
+    <child link="left_arm_base_link" />
   </joint>
   <!-- left gipper flange -->
   <link name="left_gripper_flange">
     <visual>
-      <origin xyz="0 0 0" rpy="0 0 0"/>
+      <origin xyz="0 0 0" rpy="0 0 0" />
       <geometry>
-        <mesh filename="package://ridgeback_dual_arm_description/mesh/3-finger-gripper_fixed-urdf.stl"/>
+        <mesh filename="package://ridgeback_dual_arm_description/mesh/3-finger-gripper_fixed-urdf.stl" />
       </geometry>
       <material name="">
-        <color rgba="0.2 0.2 0.2 1"/>
+        <color rgba="0.2 0.2 0.2 1" />
       </material>
     </visual>
   </link>
   <joint name="left_gripper_flange_joint" type="fixed">
-      <origin xyz="0 0 0" rpy="0 0 0"/>
-      <parent link="left_arm_tool0"/>
-      <child link="left_gripper_flange"/>
+    <origin xyz="0 0 0" rpy="0 0 0" />
+    <parent link="left_arm_tool0" />
+    <child link="left_gripper_flange" />
   </joint>
   <!-- left gripper -->
-  <xacro:robotiq-3f-gripper_articulated prefix="left_gripper_"/>
+  <xacro:robotiq-3f-gripper_articulated prefix="left_gripper_" />
   <joint name="left_gripper_joint" type="fixed">
-      <origin xyz="0 0 0.068825" rpy="${M_PI/2} 0 0"/>
-      <parent link="left_gripper_flange"/>
-      <child link="left_gripper_palm"/>
+    <origin xyz="0 0 0.068825" rpy="${M_PI/2} 0 -${M_PI/4}" />
+    <parent link="left_gripper_flange" />
+    <child link="left_gripper_palm" />
   </joint>
   <!-- right arm -->

Commit message: add dingo ur3 model

File: src/robot_description/ridgeback_dual_arm_description/urdf/ridgeback_dual_arm.urdf.xacro (robot description, xacro)
@@ -31,6 +31,6 @@
       <origin xyz="0 0 0" rpy="0 0 0" />
       <geometry>
-        <!-- <mesh filename="package://ridgeback_dual_arm_description/mesh/ridgeback_2xur5-sup-simp-urdf.stl"/> -->
-        <mesh filename="package://ridgeback_dual_arm_description/mesh/ridgeback-2xur5e-all-urdf.stl" />
+        <mesh filename="package://ridgeback_dual_arm_description/mesh/ridgeback-2xur5e-all-simp-urdf.stl"/>
+        <!-- <mesh filename="package://ridgeback_dual_arm_description/mesh/ridgeback-2xur5e-all-urdf.stl" /> -->
       </geometry>
       <material name="">

Commit message: add a table to tieta env

File: src/robot_description/ridgeback_dual_arm_description/urdf/ridgeback_dual_arm.urdf.xacro (robot description, xacro)
@@ -57,6 +57,13 @@
     <child link="left_body_link" />
   </joint>
+  <!-- left_body -->
+  <link name="right_body_link" />
+  <joint name="right_body_joint" type="fixed">
+    <origin xyz="0.2 -0.22 1.233" rpy="-${M_PI/4*3} 0 0" />
+    <parent link="base_footprint" />
+    <child link="right_body_link" />
+  </joint>
   <!-- left arm -->
-  <xacro:ur5e_robot prefix="left_arm_" />
+  <!-- <xacro:ur5e_robot prefix="left_arm_" /> -->
   <!-- <joint name="left_arm_joint" type="fixed">
       <origin xyz="0.25 0.208336 0.957336" rpy="-${M_PI/4*3} 0 0"/>
@@ -64,11 +71,11 @@
       <child link="left_arm_base_link"/>
   </joint> -->
-  <joint name="left_arm_joint" type="fixed">
+  <!-- <joint name="left_arm_joint" type="fixed">
     <origin xyz="0 0 0" rpy="${M_PI/2} ${M_PI/2} 0" />
     <parent link="left_body_link" />
     <child link="left_arm_base_link" />
-  </joint>
+  </joint> -->
   <!-- left gipper flange -->
-  <link name="left_gripper_flange">
+  <!-- <link name="left_gripper_flange">
     <visual>
       <origin xyz="0 0 0" rpy="0 0 0" />
@@ -85,21 +92,26 @@
     <parent link="left_arm_tool0" />
     <child link="left_gripper_flange" />
-  </joint>
+  </joint> -->
   <!-- left gripper -->
-  <xacro:robotiq-3f-gripper_articulated prefix="left_gripper_" />
+  <!-- <xacro:robotiq-3f-gripper_articulated prefix="left_gripper_" />
   <joint name="left_gripper_joint" type="fixed">
     <origin xyz="0 0 0.068825" rpy="${M_PI/2} 0 -${M_PI/4}" />
     <parent link="left_gripper_flange" />
     <child link="left_gripper_palm" />
-  </joint>
+  </joint> -->
   <!-- right arm -->
-  <!-- <xacro:ur5e_robot prefix="right_arm_" />
-  <joint name="right_arm_joint" type="fixed">
+  <xacro:ur5e_robot prefix="right_arm_" />
+  <!-- <joint name="right_arm_joint" type="fixed">
       <origin xyz="0.25 -0.208336 0.957336" rpy="${M_PI/4*3} 0 0"/>
       <parent link="base_footprint"/>
       <child link="right_arm_base_link"/>
   </joint> -->
+  <joint name="right_arm_joint" type="fixed">
+    <origin xyz="0 0 0" rpy="-${M_PI/2} -${M_PI/2} 0" />
+    <parent link="right_body_link" />
+    <child link="right_arm_base_link" />
+  </joint>
   <!-- right gipper flange -->
-  <!-- <link name="right_gripper_flange">
+  <link name="right_gripper_flange">
     <visual>
       <origin xyz="0 0 0" rpy="0 0 0"/>
@@ -122,11 +134,11 @@
       <parent link="right_arm_tool0"/>
       <child link="right_gripper_flange"/>
-  </joint> -->
+  </joint>
   <!-- right gripper -->
-  <!-- <xacro:robotiq-3f-gripper_articulated prefix="right_gripper_"/>
+  <xacro:robotiq-3f-gripper_articulated prefix="right_gripper_"/>
   <joint name="right_gripper_joint" type="fixed">
-      <origin xyz="0 0 0.068825" rpy="${M_PI/2} 0 0"/>
+      <origin xyz="0 0 0.068825" rpy="${M_PI/2} 0 -${M_PI/4}"/>
       <parent link="right_gripper_flange"/>
       <child link="right_gripper_palm"/>
-  </joint>   -->
+  </joint>
 </robot>

File: src/robot_description/robotiq_3f_gripper_visualization/cfg/robotiq-3f-gripper_finger_articulated_macro.xacro (robot description, xacro)
@@ -41,5 +41,5 @@
 				<material name="gray"/>
 			</visual>
-			<!-- <collision>
+			<collision>
 				<origin xyz="0.050 -.028 0" rpy="0 0 -0.52"/>
 				<geometry>
@@ -47,5 +47,5 @@
 				</geometry>
 				<material name="yellow"/>
-			</collision> -->
+			</collision>
             <inertial>
                 <origin xyz="0 0 0" rpy="0 0 0"/>

Commit message: fix tieta bodylink collision

File: src/robot_description/ridgeback_dual_arm_description/urdf/ridgeback_dual_arm.urdf.xacro (robot description, xacro)
@@ -41,5 +41,5 @@
       <origin xyz="0 0 0" rpy="0 0 0" />
       <geometry>
-        <mesh filename="package://ridgeback_dual_arm_description/mesh/ridgeback-2xur5e-all-urdf.stl" />
+        <mesh filename="package://ridgeback_dual_arm_description/mesh/ridgeback-2xur5e-all-urdf.stl" scale="1 0.5 1" />
       </geometry>
     </collision>
