Commit message: updated vicon position for tieta env

File: src/robot_description/ridgeback_description/urdf/ridgeback.urdf.xacro (robot description, xacro)
@@ -117,5 +117,5 @@
       <geometry>
         <!-- <mesh filename="package://ridgeback_description/meshes/body-collision.stl"/> -->
-        <box size="0.95 0.8 0.3"/>
+        <box size="0.95 0.8 0.5"/>
       </geometry>
     </collision>

Commit message: added base_link collision for astar

File: src/robot_description/ridgeback_description/urdf/ridgeback.urdf.xacro (robot description, xacro)
@@ -99,5 +99,13 @@
     <limit effort="0" velocity="0" />
   </xacro:rocker>
-  <link name="base_link"></link>
+  <link name="base_link">
+      <collision>
+      <origin xyz="0 0 0.15"/>
+      <geometry>
+        <!-- <mesh filename="package://ridgeback_description/meshes/body-collision.stl"/> -->
+        <box size="0.95 0.8 0.5"/>
+      </geometry>
+    </collision>
+    </link>
   <joint name="base_link_joint" type="fixed">
     <origin xyz="0 0 0" rpy="0 0 0" />
@@ -113,11 +121,4 @@
       <material name="black" />
     </visual>
-    <collision>
-      <origin xyz="0 0 0.15"/>
-      <geometry>
-        <!-- <mesh filename="package://ridgeback_description/meshes/body-collision.stl"/> -->
-        <box size="0.95 0.8 0.5"/>
-      </geometry>
-    </collision>
     <inertial>
       <origin xyz="0.012 0.002 0.067" rpy="${PI/2} 0 ${PI/2}"/>
