Commit message: finish exp 4

File: src/vkc_example/urdf/deploy_husky_ur5e_2f_85.urdf.xacro (robot description, xacro)
@@ -18,5 +18,5 @@
       <child link="base_link" />
       <axis xyz="0 0 1" />
-      <limit effort="20" velocity="5.0" lower="-6.28" upper="6.28" />
+      <limit effort="20" velocity="5.0" lower="-3.14" upper="3.14" />
     </joint>
     <joint name="${prefix}base_theta_base_y" type="prismatic">
